File: esp32s3-microsd-devkit.kicad_sch (KiCad schematic)
At the start: 9 parts, among them J1 Conn_01x17, J3 Conn_01x17, U1 ESP32-S3-WROOM-1

Commit message: Fix cross-wired USB lines
Connections:
- net USB C/USB_D+: now also U1.14 (IO20); no longer U1.13 (IO19)
- net USB C/USB_D-: now also U1.13 (IO19); no longer U1.14 (IO20)
Changed lines of the file:
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@@
+    (stroke (width 0) (type default))
+  )
+  (wire (pts (xy 113.03 74.93) (xy 140.97 74.93))
+    (stroke (width 0) (type default))
+  )
+  (wire (pts (xy 135.89 26.67) (xy 142.24 26.67))
+    (stroke (width 0) (type default))
+  )
+  (wire (pts (xy 194.31 74.93) (xy 196.85 74.93))
+    (stroke (width 0) (type default))
+  )
+  (wire (pts (xy 247.65 115.57) (xy 265.43 115.57))
+    (stroke (width 0) (type default))
+  )
+  (wire (pts (xy 247.65 120.65) (xy 265.43 120.65))
+    (stroke (width 0) (type default))
+  )
+  (wire (pts (xy 247.65 92.71) (xy 265.43 92.71))
+    (stroke (width 0) (type default))
+  )
+  (wire (pts (xy 104.14 87.63) (xy 140.97 87.63))
+    (stroke (width 0) (type default))
+  )
+  (wire (pts (xy 102.87 97.79) (xy 140.97 97.79))
+    (stroke (width 0) (type default))
+  )
+  (wire (pts (xy 171.45 105.41) (xy 187.96 105.41))
+    (stroke (width 0) (type default))
+  )
+  (wire (pts (xy 171.45 97.79) (xy 187.96 97.79))
+    (stroke (width 0) (type default))
+  )
+  (wire (pts (xy 173.99 55.88) (xy 173.99 72.39))
+    (stroke (width 0) (type default))
+  )
+  (wire (pts (xy 171.45 92.71) (xy 208.28 92.71))
+    (stroke (width 0) (type default))
+  )
+  (wire (pts (xy 194.31 67.31) (xy 194.31 74.93))
+    (stroke (width 0) (type default))
+  )
+  (wire (pts (xy 102.87 125.73) (xy 140.97 125.73))
+    (stroke (width 0) (type default))
+  )
+  (wire (pts (xy 247.65 113.03) (xy 265.43 113.03))
     (stroke (width 0) (type default))
   )
@@
     (stroke (width 0) (type default))
   )
-  (wire (pts (xy 113.03 74.93) (xy 140.97 74.93))
-    (stroke (width 0) (type default))
-  )
-  (wire (pts (xy 135.89 26.67) (xy 142.24 26.67))
-    (stroke (width 0) (type default))
-  )
-  (wire (pts (xy 194.31 74.93) (xy 196.85 74.93))
-    (stroke (width 0) (type default))
-  )
-  (wire (pts (xy 247.65 115.57) (xy 265.43 115.57))
-    (stroke (width 0) (type default))
-  )
-  (wire (pts (xy 247.65 120.65) (xy 265.43 120.65))
-    (stroke (width 0) (type default))
-  )
-  (wire (pts (xy 247.65 92.71) (xy 265.43 92.71))
-    (stroke (width 0) (type default))
-  )
-  (wire (pts (xy 104.14 87.63) (xy 140.97 87.63))
-    (stroke (width 0) (type default))
-  )
-  (wire (pts (xy 102.87 97.79) (xy 140.97 97.79))
-    (stroke (width 0) (type default))
-  )
-  (wire (pts (xy 171.45 105.41) (xy 187.96 105.41))
-    (stroke (width 0) (type default))
-  )
-  (wire (pts (xy 171.45 97.79) (xy 187.96 97.79))
-    (stroke (width 0) (type default))
-  )
-  (wire (pts (xy 173.99 55.88) (xy 173.99 72.39))
-    (stroke (width 0) (type default))
-  )
-  (wire (pts (xy 194.31 67.31) (xy 194.31 74.93))
-    (stroke (width 0) (type default))
-  )
-  (wire (pts (xy 102.87 125.73) (xy 140.97 125.73))
-    (stroke (width 0) (type default))
-  )
-  (wire (pts (xy 247.65 113.03) (xy 265.43 113.03))
-    (stroke (width 0) (type default))
-  )
   (wire (pts (xy 247.65 90.17) (xy 265.43 90.17))
     (stroke (width 0) (type default))
@@
   )
   (wire (pts (xy 115.57 95.25) (xy 140.97 95.25))
-    (stroke (width 0) (type default))
-  )
-  (wire (pts (xy 171.45 92.71) (xy 208.28 92.71))
     (stroke (width 0) (type default))
   )
@@
       (effects (font (size 1.27 1.27)) (justify left top))
     )
-    (pin "USB_D+" input (at 208.28 92.71 180)
-      (effects (font (size 1.27 1.27)) (justify left))
-    )
-    (pin "USB_D-" input (at 208.28 95.25 180)
-      (effects (font (size 1.27 1.27)) (justify left))
-    )
+    (pin "USB_D+" input (at 208.28 95.25 180)
+      (effects (font (size 1.27 1.27)) (justify left))
+    )
+    (pin "USB_D-" input (at 208.28 92.71 180)
+      (effects (font (size 1.27 1.27)) (justify left))
+    )
