File: usb_c.kicad_sch (KiCad schematic)
At the start: 10 parts, among them J2 USB4105-GF-A, U2 USBLC6-2P6, U3 MIC23150-SYMT-TR

Commit message: Ready to make v0.1
Parts:
- added D2: B0540WS-TP, Diode_SMD:D_SOD-123, symbol downloaded_parts:MBR230LS
- added H1, H2, H3: MountingHole, MountingHole:MountingHole_2.2mm_M2_ISO7380_Pad, symbol Mechanical:MountingHole
- added TP1, TP2, TP3: TestPoint, TestPoint:TestPoint_Pad_1.5x1.5mm, symbol Connector:TestPoint
Connections:
- net +3.3V: now also TP1.1
- net +5V: now also D2.1 (K), TP2.1; no longer J2.A4 (VBUS), J2.A9 (VBUS), J2.B4 (VBUS), J2.B9 (VBUS)
- net GND: now also TP3.1
- new net: D2.2 (A), J2.A4 (VBUS), J2.A9 (VBUS), J2.B4 (VBUS), J2.B9 (VBUS)
Changed lines of the file:
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@@
   (junction (at 73.66 107.95) (diameter 0) (color 0 0 0 0)
+  )
+  (junction (at 160.02 129.54) (diameter 0) (color 0 0 0 0)
   )
   (junction (at 189.23 140.97) (diameter 0) (color 0 0 0 0)
@@
     (stroke (width 0) (type default))
   )
+  (wire (pts (xy 105.41 39.37) (xy 120.65 39.37))
+    (stroke (width 0) (type default))
+  )
   (wire (pts (xy 106.68 46.99) (xy 127 46.99))
     (stroke (width 0) (type default))
   )
+  (wire (pts (xy 240.03 118.11) (xy 240.03 123.19))
+    (stroke (width 0) (type default))
+  )
   (wire (pts (xy 179.07 57.15) (xy 179.07 58.42))
     (stroke (width 0) (type default))
@@
     (stroke (width 0) (type default))
   )
-  (wire (pts (xy 88.9 39.37) (xy 120.65 39.37))
+  (wire (pts (xy 88.9 39.37) (xy 100.33 39.37))
     (stroke (width 0) (type default))
   )
@@
     (stroke (width 0) (type default))
   )
-  (wire (pts (xy 154.94 129.54) (xy 166.37 129.54))
+  (wire (pts (xy 154.94 129.54) (xy 160.02 129.54))
     (stroke (width 0) (type default))
   )
@@
     (stroke (width 0) (type default))
   )
+  (wire (pts (xy 240.03 140.97) (xy 240.03 148.59))
+    (stroke (width 0) (type default))
+  )
   (wire (pts (xy 198.12 123.19) (xy 201.93 123.19))
     (stroke (width 0) (type default))
@@
     (stroke (width 0) (type default))
   )
+  (wire (pts (xy 160.02 129.54) (xy 166.37 129.54))
+    (stroke (width 0) (type default))
+  )
   (wire (pts (xy 186.69 135.89) (xy 186.69 140.97))
     (stroke (width 0) (type default))
@@
   )
   (wire (pts (xy 186.69 140.97) (xy 189.23 140.97))
+    (stroke (width 0) (type default))
+  )
+  (wire (pts (xy 160.02 119.38) (xy 160.02 129.54))
     (stroke (width 0) (type default))
   )
@@
         (path "/2052380c-6188-4155-bdc5-6e5f1a2703a4/59878365-3733-4c42-8ae0-148d66fa8c40"
           (reference "#PWR019") (unit 1)
+        )
+      )
+    )
+  )
+  (symbol (lib_id "Mechanical:MountingHole") (at 31.75 66.04 0) (unit 1)
+    (in_bom yes) (on_board yes) (dnp no) (fields_autoplaced)
+    (property "Reference" "H1" (at 34.29 64.77 0)
+      (effects (font (size 1.27 1.27)) (justify left))
+    )
+    (property "Value" "MountingHole" (at 34.29 67.31 0)
+      (effects (font (size 1.27 1.27)) (justify left))
+    )
+    (property "Footprint" "MountingHole:MountingHole_2.2mm_M2_ISO7380_Pad" (at 31.75 66.04 0)
+      (effects (font (size 1.27 1.27)) hide)
+    )
+    (property "Datasheet" "~" (at 31.75 66.04 0)
+      (effects (font (size 1.27 1.27)) hide)
+    )
+    (instances
+      (project "esp32s3-microsd-devkit"
+        (path "/2052380c-6188-4155-bdc5-6e5f1a2703a4/59878365-3733-4c42-8ae0-148d66fa8c40"
+          (reference "H1") (unit 1)
+        )
+      )
+    )
+  )
+  (symbol (lib_id "Connector:TestPoint") (at 240.03 118.11 0) (unit 1)
+    (in_bom yes) (on_board yes) (dnp no) (fields_autoplaced)
+    (property "Reference" "TP1" (at 242.57 113.538 0)
+      (effects (font (size 1.27 1.27)) (justify left))
+    )
+    (property "Value" "TestPoint" (at 242.57 116.078 0)
+      (effects (font (size 1.27 1.27)) (justify left))
+    )
+    (property "Footprint" "TestPoint:TestPoint_Pad_1.5x1.5mm" (at 245.11 118.11 0)
+      (effects (font (size 1.27 1.27)) hide)
+    )
+    (property "Datasheet" "~" (at 245.11 118.11 0)
+      (effects (font (size 1.27 1.27)) hide)
+    )
+    (pin "1")
+    (instances
+      (project "esp32s3-microsd-devkit"
+        (path "/2052380c-6188-4155-bdc5-6e5f1a2703a4/59878365-3733-4c42-8ae0-148d66fa8c40"
+          (reference "TP1") (unit 1)
         )
       )
@@
     )
   )
+  (symbol (lib_id "Connector:TestPoint") (at 240.03 148.59 180) (unit 1)
+    (in_bom yes) (on_board yes) (dnp no) (fields_autoplaced)
+    (property "Reference" "TP3" (at 242.57 150.622 0)
+      (effects (font (size 1.27 1.27)) (justify right))
+    )
+    (property "Value" "TestPoint" (at 242.57 153.162 0)
+      (effects (font (size 1.27 1.27)) (justify right))
+    )
+    (property "Footprint" "TestPoint:TestPoint_Pad_1.5x1.5mm" (at 234.95 148.59 0)
+      (effects (font (size 1.27 1.27)) hide)
+    )
+    (property "Datasheet" "~" (at 234.95 148.59 0)
+      (effects (font (size 1.27 1.27)) hide)
+    )
+    (pin "1")
+    (instances
+      (project "esp32s3-microsd-devkit"
+        (path "/2052380c-6188-4155-bdc5-6e5f1a2703a4/59878365-3733-4c42-8ae0-148d66fa8c40"
+          (reference "TP3") (unit 1)
+        )
+      )
+    )
+  )
+  (symbol (lib_id "Connector:TestPoint") (at 160.02 119.38 0) (unit 1)
+    (in_bom yes) (on_board yes) (dnp no) (fields_autoplaced)
+    (property "Reference" "TP2" (at 162.56 114.808 0)
+      (effects (font (size 1.27 1.27)) (justify left))
+    )
+    (property "Value" "TestPoint" (at 162.56 117.348 0)
+      (effects (font (size 1.27 1.27)) (justify left))
+    )
+    (property "Footprint" "TestPoint:TestPoint_Pad_1.5x1.5mm" (at 165.1 119.38 0)
+      (effects (font (size 1.27 1.27)) hide)
+    )
+    (property "Datasheet" "~" (at 165.1 119.38 0)
+      (effects (font (size 1.27 1.27)) hide)
+    )
+    (pin "1")
+    (instances
+      (project "esp32s3-microsd-devkit"
+        (path "/2052380c-6188-4155-bdc5-6e5f1a2703a4/59878365-3733-4c42-8ae0-148d66fa8c40"
+          (reference "TP2") (unit 1)
+        )
+      )
+    )
+  )
   (symbol (lib_id "power:+5V") (at 154.94 129.54 90) (unit 1)
     (in_bom yes) (on_board yes) (dnp no) (fields_autoplaced)
@@
         (path "/c0262c8b-3aa0-4ed4-b708-90fc6d37b827/0aeec02c-19c9-480f-8f4e-3e0e4857ed79"
           (reference "#PWR08") (unit 1)
+        )
+      )
+    )
+  )
+  (symbol (lib_id "Mechanical:MountingHole") (at 31.75 40.64 0) (unit 1)
+    (in_bom yes) (on_board yes) (dnp no) (fields_autoplaced)
+    (property "Reference" "H2" (at 34.29 39.37 0)
+      (effects (font (size 1.27 1.27)) (justify left))
+    )
+    (property "Value" "MountingHole" (at 34.29 41.91 0)
+      (effects (font (size 1.27 1.27)) (justify left))
+    )
+    (property "Footprint" "MountingHole:MountingHole_2.2mm_M2_ISO7380_Pad" (at 31.75 40.64 0)
+      (effects (font (size 1.27 1.27)) hide)
+    )
+    (property "Datasheet" "~" (at 31.75 40.64 0)
+      (effects (font (size 1.27 1.27)) hide)
+    )
+    (instances
+      (project "esp32s3-microsd-devkit"
+        (path "/2052380c-6188-4155-bdc5-6e5f1a2703a4/59878365-3733-4c42-8ae0-148d66fa8c40"
+          (reference "H2") (unit 1)
         )
       )
@@
         (path "/c0262c8b-3aa0-4ed4-b708-90fc6d37b827/0aeec02c-19c9-480f-8f4e-3e0e4857ed79"
           (reference "C2") (unit 1)
+        )
+      )
+    )
+  )
+  (symbol (lib_id "downloaded_parts:MBR230LS") (at 102.87 39.37 180) (unit 1)
+    (in_bom yes) (on_board yes) (dnp no) (fields_autoplaced)
+    (property "Reference" "D2" (at 103.124 35.56 0)
+      (effects (font (size 1.27 1.27)))
+    )
+    (property "Value" "B0540WS-TP" (at 109.22 33.02 0)
+      (effects (font (size 1.27 1.27)) (justify left) hide)
+    )
+    (property "Footprint" "Diode_SMD:D_SOD-123" (at 102.87 30.48 0)
+      (effects (font (size 1.27 1.27)) hide)
+    )
+    (property "Datasheet" "https://www.smc-diodes.com/propdf/MBR230LS%20N1466%20REV.A.pdf" (at 102.87 27.94 0)
+      (effects (font (size 1.27 1.27)) hide)
+    )
+    (property "Forward Voltage" "500mV" (at 102.87 35.56 0)
+      (effects (font (size 1.27 1.27)) hide)
+    )
+    (property "Current" "2A" (at 97.79 35.56 0)
+      (effects (font (size 1.27 1.27)) hide)
+    )
+    (property "Voltage" "40V" (at 111.76 35.56 0)
+      (effects (font (size 1.27 1.27)) hide)
+    )
+    (property "Reverse Voltage" "30V" (at 109.22 35.56 0)
+      (effects (font (size 1.27 1.27)) hide)
+    )
+    (pin "1")
+    (pin "2")
+    (instances
+      (project "esp32s3-microsd-devkit"
+        (path "/2052380c-6188-4155-bdc5-6e5f1a2703a4/59878365-3733-4c42-8ae0-148d66fa8c40"
+          (reference "D2") (unit 1)
         )
       )
@@
         )
       )
+    )
+  )
+  (symbol (lib_id "Mechanical:MountingHole") (at 31.75 49.53 0) (unit 1)
+    (in_bom yes) (on_board yes) (dnp no) (fields_autoplaced)
+    (property "Reference" "H3" (at 34.29 48.26 0)
+      (effects (font (size 1.27 1.27)) (justify left))
+    )
+    (property "Value" "MountingHole" (at 34.29 50.8 0)
+      (effects (font (size 1.27 1.27)) (justify left))
+    )
+    (property "Footprint" "MountingHole:MountingHole_2.2mm_M2_ISO7380_Pad" (at 31.75 49.53 0)
+      (effects (font (size 1.27 1.27)) hide)
+    )
+    (property "Datasheet" "~" (at 31.75 49.53 0)
+      (effects (font (size 1.27 1.27)) hide)
+    )
+    (instances
+      (project "esp32s3-microsd-devkit"
+        (path "/2052380c-6188-4155-bdc5-6e5f1a2703a4/59878365-3733-4c42-8ae0-148d66fa8c40"
+          (reference "H3") (unit 1)
+        )
+      )

Commit message: Fix diode part number
Parts:
- D2: value B0540WS-TP -> MBR230LS
Changed lines of the file:
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@@
       (effects (font (size 1.27 1.27)))
     )
-    (property "Value" "B0540WS-TP" (at 109.22 33.02 0)
+    (property "Value" "MBR230LS" (at 109.22 33.02 0)
       (effects (font (size 1.27 1.27)) (justify left) hide)
     )
